File: Labs/04-interrupts/KnightRider/KnightRider.sch (KiCad schematic (older format))
At the start: 12 parts, among them SW1 SW_Push

Commit message: readme
Parts:
- removed D3: CQY99, LED_THT:LED_D5.0mm_IRGrey, symbol LED:CQY99
- removed R1: 510, symbol Device:R
- added A?: Arduino_UNO_R3, Module:Arduino_UNO_R3, symbol MCU_Module:Arduino_UNO_R3
- added D?: CQY99, LED_THT:LED_D5.0mm_IRGrey, symbol LED:CQY99
- added R?: 510, symbol Device:R
- added SW?: SW_Push, symbol Switch:SW_Push
Connections:
- net +5V: now also A?.5 (+5V)
- net GND: now also A?.29 (GND), A?.6 (GND), A?.7 (GND), D?.1 (K), SW?.1
- net at A1.10 (A1): now also SW1.2
- net at A1.9 (A0): no longer SW1.2
- new net: A?.10 (A1), SW?.2
- new net: A?.28 (D13), R?.1
- new net: D?.2 (A), R?.2
Other:
- moved on the sheet: SW1
Changed lines of the file:
@@
 L Switch:SW_Push SW1
 U 1 1 61550227
-P 5700 3550
-F 0 "SW1" H 5700 3835 50  0000 C CNN
-F 1 "SW_Push" H 5700 3744 50  0000 C CNN
-F 2 "" H 5700 3750 50  0001 C CNN
-F 3 "~" H 5700 3750 50  0001 C CNN
-	1    5700 3550
+P 5700 3650
+F 0 "SW1" H 5700 3935 50  0000 C CNN
+F 1 "SW_Push" H 5700 3844 50  0000 C CNN
+F 2 "" H 5700 3850 50  0001 C CNN
+F 3 "~" H 5700 3850 50  0001 C CNN
+	1    5700 3650
 	-1   0    0    -1
 $EndComp
@@
 L power:GND #PWR02
 U 1 1 61551592
-P 6000 3700
-F 0 "#PWR02" H 6000 3450 50  0001 C CNN
-F 1 "GND" H 6005 3527 50  0000 C CNN
-F 2 "" H 6000 3700 50  0001 C CNN
-F 3 "" H 6000 3700 50  0001 C CNN
-	1    6000 3700
+P 6000 3800
+F 0 "#PWR02" H 6000 3550 50  0001 C CNN
+F 1 "GND" H 6005 3627 50  0000 C CNN
+F 2 "" H 6000 3800 50  0001 C CNN
+F 3 "" H 6000 3800 50  0001 C CNN
+	1    6000 3800
 	-1   0    0    -1
 $EndComp
@@
 $EndComp
 $Comp
-L Device:R R1
-U 1 1 6155D8E1
-P 3400 3750
-F 0 "R1" V 3193 3750 50  0000 C CNN
-F 1 "510" V 3284 3750 50  0000 C CNN
-F 2 "" V 3330 3750 50  0001 C CNN
-F 3 "~" H 3400 3750 50  0001 C CNN
-	1    3400 3750
-	0    1    1    0
-$EndComp
-$Comp
 L LED:CQY99 D4
 U 1 1 61561493
@@
 	1    0    0    -1
 $EndComp
-$Comp
-L LED:CQY99 D3
-U 1 1 6157629A
-P 3000 3750
-F 0 "D3" H 2950 4040 50  0000 C CNN
-F 1 "CQY99" H 2950 3949 50  0000 C CNN
-F 2 "LED_THT:LED_D5.0mm_IRGrey" H 3000 3925 50  0001 C CNN
-F 3 "https://www.prtice.info/IMG/pdf/CQY99.pdf" H 2950 3750 50  0001 C CNN
-	1    3000 3750
-	1    0    0    -1
-$EndComp
-Wire Wire Line
-	3250 3750 3100 3750
 Wire Wire Line
 	3250 4100 2850 4100
@@
 	3250 5150 3100 5150
 Wire Wire Line
-	2800 3750 2000 3750
-Wire Wire Line
 	2550 4100 2000 4100
 Wire Wire Line
-	2000 4100 2000 3750
-Wire Wire Line
 	2800 4450 2000 4450
 Wire Wire Line
 	2000 4450 2000 4100
-Connection ~ 2000 4100
 Wire Wire Line
 	2550 4800 2000 4800
@@
 	3650 4100 3550 4100
 Wire Wire Line
-	3950 3850 3650 3850
-Wire Wire Line
-	3650 3850 3650 3750
-Wire Wire Line
-	3650 3750 3550 3750
-Wire Wire Line
-	4950 3550 5500 3550
-Wire Wire Line
-	5900 3550 6000 3550
-Wire Wire Line
-	6000 3550 6000 3700
+	4950 3650 5500 3650
+Wire Wire Line
+	5900 3650 6000 3650
+Wire Wire Line
+	6000 3650 6000 3800
+$Comp
+L MCU_Module:Arduino_UNO_R3 A?
+U 1 1 61686606
+P 9100 3350
+F 0 "A?" H 8550 4450 50  0000 C CNN
+F 1 "Arduino_UNO_R3" H 8550 4350 50  0000 C CNN
+F 2 "Module:Arduino_UNO_R3" H 9100 3350 50  0001 C CIN
+F 3 "https://www.arduino.cc/en/Main/arduinoBoardUno" H 9100 3350 50  0001 C CNN
+	1    9100 3350
+	1    0    0    -1
+$EndComp
+$Comp
+L power:GND #PWR?
+U 1 1 6168660C
+P 9100 4800
+F 0 "#PWR?" H 9100 4550 50  0001 C CNN
+F 1 "GND" H 9105 4627 50  0000 C CNN
+F 2 "" H 9100 4800 50  0001 C CNN
+F 3 "" H 9100 4800 50  0001 C CNN
+	1    9100 4800
+	1    0    0    -1
+$EndComp
+Wire Wire Line
+	9000 4450 9000 4650
+Wire Wire Line
+	9000 4650 9100 4650
+Wire Wire Line
+	9100 4650 9100 4800
+Wire Wire Line
+	9200 4450 9200 4650
+Wire Wire Line
+	9200 4650 9100 4650
+Connection ~ 9100 4650
+Wire Wire Line
+	9100 4450 9100 4650
+$Comp
+L power:+5V #PWR?
+U 1 1 61686619
+P 9300 2200
+F 0 "#PWR?" H 9300 2050 50  0001 C CNN
+F 1 "+5V" H 9315 2373 50  0000 C CNN
+F 2 "" H 9300 2200 50  0001 C CNN
+F 3 "" H 9300 2200 50  0001 C CNN
+	1    9300 2200
+	1    0    0    -1
+$EndComp
+Wire Wire Line
+	9300 2200 9300 2350
+$Comp
+L Switch:SW_Push SW?
+U 1 1 61686626
+P 10350 3450
+F 0 "SW?" H 10350 3735 50  0000 C CNN
+F 1 "SW_Push" H 10350 3644 50  0000 C CNN
+F 2 "" H 10350 3650 50  0001 C CNN
+F 3 "~" H 10350 3650 50  0001 C CNN
+	1    10350 3450
+	-1   0    0    -1
+$EndComp
+$Comp
+L power:GND #PWR?
+U 1 1 6168662C
+P 10650 3600
+F 0 "#PWR?" H 10650 3350 50  0001 C CNN
+F 1 "GND" H 10655 3427 50  0000 C CNN
+F 2 "" H 10650 3600 50  0001 C CNN
+F 3 "" H 10650 3600 50  0001 C CNN
+	1    10650 3600
+	-1   0    0    -1
+$EndComp
+$Comp
+L LED:CQY99 D?
+U 1 1 61686638
+P 7750 4050
+F 0 "D?" H 7700 4340 50  0000 C CNN
+F 1 "CQY99" H 7700 4249 50  0000 C CNN
+F 2 "LED_THT:LED_D5.0mm_IRGrey" H 7750 4225 50  0001 C CNN
+F 3 "https://www.prtice.info/IMG/pdf/CQY99.pdf" H 7700 4050 50  0001 C CNN
+	1    7750 4050
+	1    0    0    -1
+$EndComp
+$Comp
+L Device:R R?
+U 1 1 6168664A
+P 8200 4050
+F 0 "R?" V 7993 4050 50  0000 C CNN
+F 1 "510" V 8084 4050 50  0000 C CNN
+F 2 "" V 8130 4050 50  0001 C CNN
+F 3 "~" H 8200 4050 50  0001 C CNN
+	1    8200 4050
+	0    1    1    0
+$EndComp
+$Comp
+L power:GND #PWR?
+U 1 1 61686669
+P 7350 4150
+F 0 "#PWR?" H 7350 3900 50  0001 C CNN
+F 1 "GND" H 7355 3977 50  0000 C CNN
+F 2 "" H 7350 4150 50  0001 C CNN
+F 3 "" H 7350 4150 50  0001 C CNN
+	1    7350 4150
+	1    0    0    -1
+$EndComp
+Wire Wire Line
+	9600 3450 10150 3450
+Wire Wire Line
+	10550 3450 10650 3450
+Wire Wire Line
+	10650 3450 10650 3600
+Wire Wire Line
+	8350 4050 8600 4050
+Wire Wire Line
+	8050 4050 7850 4050
+Wire Wire Line
+	7550 4050 7350 4050
+Wire Wire Line
+	7350 4050 7350 4150
 $EndSCHEMATC

Commit message: readme
Parts:
- removed A?: Arduino_UNO_R3, Module:Arduino_UNO_R3, symbol MCU_Module:Arduino_UNO_R3
- removed D1, D2, D4, D5, D?: CQY99, LED_THT:LED_D5.0mm_IRGrey, symbol LED:CQY99
- removed R5, R?: 510, symbol Device:R
- removed SW?: SW_Push, symbol Switch:SW_Push
- added D1, D2, D3, D4: LED, symbol Device:LED
- added R2: 1k, symbol Device:R
- R1: renamed from R2; value 510 -> 1k
- R3, R4: value 510 -> 1k
Connections:
- net +5V: now also D1.2 (A), D2.2 (A), D3.2 (A), D4.2 (A)
- net at A1.26 (D11): now also R2.1; no longer R3.1
- net at A1.27 (D12): now also R3.1; no longer R4.1
- net at A1.28 (D13): now also R4.1
- net at R1.2: now also D4.1 (K)
- net at R4.2: now also D1.1 (K)
- net at R3.2: now also D2.1 (K)
- new net: D3.1 (K), R2.2
Changed lines of the file:
@@
 	4450 4650 4450 4850
 $Comp
-L power:+5V #PWR04
+L power:+5V #PWR01
 U 1 1 6154D3B6
 P 4650 2400
-F 0 "#PWR04" H 4650 2250 50  0001 C CNN
+F 0 "#PWR01" H 4650 2250 50  0001 C CNN
 F 1 "+5V" H 4665 2573 50  0000 C CNN
 F 2 "" H 4650 2400 50  0001 C CNN
@@
 Wire Wire Line
 	4650 2400 4650 2550
-$Comp
-L LED:CQY99 D1
-U 1 1 6154F463
-P 2750 4100
-F 0 "D1" H 2700 4390 50  0000 C CNN
-F 1 "CQY99" H 2700 4299 50  0000 C CNN
-F 2 "LED_THT:LED_D5.0mm_IRGrey" H 2750 4275 50  0001 C CNN
-F 3 "https://www.prtice.info/IMG/pdf/CQY99.pdf" H 2700 4100 50  0001 C CNN
-	1    2750 4100
-	1    0    0    -1
-$EndComp
 $Comp
 L Switch:SW_Push SW1
@@
 $EndComp
 $Comp
-L LED:CQY99 D2
-U 1 1 61552C59
-P 2750 4800
-F 0 "D2" H 2700 5090 50  0000 C CNN
-F 1 "CQY99" H 2700 4999 50  0000 C CNN
-F 2 "LED_THT:LED_D5.0mm_IRGrey" H 2750 4975 50  0001 C CNN
-F 3 "https://www.prtice.info/IMG/pdf/CQY99.pdf" H 2700 4800 50  0001 C CNN
-	1    2750 4800
-	1    0    0    -1
-$EndComp
-$Comp
-L LED:CQY99 D5
-U 1 1 6155303B
-P 3000 5150
-F 0 "D5" H 2950 5440 50  0000 C CNN
-F 1 "CQY99" H 2950 5349 50  0000 C CNN
-F 2 "LED_THT:LED_D5.0mm_IRGrey" H 3000 5325 50  0001 C CNN
-F 3 "https://www.prtice.info/IMG/pdf/CQY99.pdf" H 2950 5150 50  0001 C CNN
-	1    3000 5150
-	1    0    0    -1
-$EndComp
-$Comp
-L Device:R R3
-U 1 1 61553F38
-P 3400 4450
-F 0 "R3" V 3193 4450 50  0000 C CNN
-F 1 "510" V 3284 4450 50  0000 C CNN
-F 2 "" V 3330 4450 50  0001 C CNN
-F 3 "~" H 3400 4450 50  0001 C CNN
-	1    3400 4450
-	0    1    1    0
-$EndComp
-$Comp
-L Device:R R4
-U 1 1 61554B16
-P 3400 4800
-F 0 "R4" V 3193 4800 50  0000 C CNN
-F 1 "510" V 3284 4800 50  0000 C CNN
-F 2 "" V 3330 4800 50  0001 C CNN
-F 3 "~" H 3400 4800 50  0001 C CNN
-	1    3400 4800
-	0    1    1    0
-$EndComp
-$Comp
-L Device:R R5
-U 1 1 61554FCB
-P 3400 5150
-F 0 "R5" V 3193 5150 50  0000 C CNN
-F 1 "510" V 3284 5150 50  0000 C CNN
-F 2 "" V 3330 5150 50  0001 C CNN
-F 3 "~" H 3400 5150 50  0001 C CNN
-	1    3400 5150
-	0    1    1    0
-$EndComp
-$Comp
-L Device:R R2
+L Device:R R1
 U 1 1 6155CCC8
 P 3400 4100
-F 0 "R2" V 3193 4100 50  0000 C CNN
-F 1 "510" V 3284 4100 50  0000 C CNN
+F 0 "R1" V 3193 4100 50  0000 C CNN
+F 1 "1k" V 3284 4100 50  0000 C CNN
 F 2 "" V 3330 4100 50  0001 C CNN
 F 3 "~" H 3400 4100 50  0001 C CNN
@@
 	0    1    1    0
 $EndComp
-$Comp
-L LED:CQY99 D4
-U 1 1 61561493
-P 3000 4450
-F 0 "D4" H 2950 4740 50  0000 C CNN
-F 1 "CQY99" H 2950 4649 50  0000 C CNN
-F 2 "LED_THT:LED_D5.0mm_IRGrey" H 3000 4625 50  0001 C CNN
-F 3 "https://www.prtice.info/IMG/pdf/CQY99.pdf" H 2950 4450 50  0001 C CNN
-	1    3000 4450
-	1    0    0    -1
-$EndComp
-Wire Wire Line
-	3250 4100 2850 4100
 Wire Wire Line
 	3250 4450 3100 4450
@@
 Wire Wire Line
 	2550 4100 2000 4100
-Wire Wire Line
-	2800 4450 2000 4450
 Wire Wire Line
 	2000 4450 2000 4100
@@
 	2000 5150 2000 4800
 Connection ~ 2000 4800
-$Comp
-L power:GND #PWR01
-U 1 1 6158368D
-P 2000 5350
-F 0 "#PWR01" H 2000 5100 50  0001 C CNN
-F 1 "GND" H 2005 5177 50  0000 C CNN
-F 2 "" H 2000 5350 50  0001 C CNN
-F 3 "" H 2000 5350 50  0001 C CNN
-	1    2000 5350
-	1    0    0    -1
-$EndComp
-Wire Wire Line
-	2000 5350 2000 5150
-Connection ~ 2000 5150
 Wire Wire Line
 	3950 4250 3900 4250
@@
 	6000 3650 6000 3800
 $Comp
-L MCU_Module:Arduino_UNO_R3 A?
-U 1 1 61686606
-P 9100 3350
-F 0 "A?" H 8550 4450 50  0000 C CNN
-F 1 "Arduino_UNO_R3" H 8550 4350 50  0000 C CNN
-F 2 "Module:Arduino_UNO_R3" H 9100 3350 50  0001 C CIN
-F 3 "https://www.arduino.cc/en/Main/arduinoBoardUno" H 9100 3350 50  0001 C CNN
-	1    9100 3350
-	1    0    0    -1
+L Device:R R2
+U 1 1 616EC87C
+P 3400 4450
+F 0 "R2" V 3193 4450 50  0000 C CNN
+F 1 "1k" V 3284 4450 50  0000 C CNN
+F 2 "" V 3330 4450 50  0001 C CNN
+F 3 "~" H 3400 4450 50  0001 C CNN
+	1    3400 4450
+	0    1    1    0
 $EndComp
 $Comp
-L power:GND #PWR?
-U 1 1 6168660C
-P 9100 4800
-F 0 "#PWR?" H 9100 4550 50  0001 C CNN
-F 1 "GND" H 9105 4627 50  0000 C CNN
-F 2 "" H 9100 4800 50  0001 C CNN
-F 3 "" H 9100 4800 50  0001 C CNN
-	1    9100 4800
+L Device:R R3
+U 1 1 616ECB37
+P 3400 4800
+F 0 "R3" V 3193 4800 50  0000 C CNN
+F 1 "1k" V 3284 4800 50  0000 C CNN
+F 2 "" V 3330 4800 50  0001 C CNN
+F 3 "~" H 3400 4800 50  0001 C CNN
+	1    3400 4800
+	0    1    1    0
+$EndComp
+$Comp
+L Device:R R4
+U 1 1 616ECDF3
+P 3400 5150
+F 0 "R4" V 3193 5150 50  0000 C CNN
+F 1 "1k" V 3284 5150 50  0000 C CNN
+F 2 "" V 3330 5150 50  0001 C CNN
+F 3 "~" H 3400 5150 50  0001 C CNN
+	1    3400 5150
+	0    1    1    0
+$EndComp
+$Comp
+L power:+5V #PWR?
+U 1 1 616EF1B9
+P 2000 3950
+F 0 "#PWR?" H 2000 3800 50  0001 C CNN
+F 1 "+5V" H 2015 4123 50  0000 C CNN
+F 2 "" H 2000 3950 50  0001 C CNN
+F 3 "" H 2000 3950 50  0001 C CNN
+	1    2000 3950
 	1    0    0    -1
 $EndComp
 Wire Wire Line
-	9000 4450 9000 4650
+	2000 4100 2000 3950
+Connection ~ 2000 4100
 Wire Wire Line
-	9000 4650 9100 4650
-Wire Wire Line
-	9100 4650 9100 4800
-Wire Wire Line
-	9200 4450 9200 4650
-Wire Wire Line
-	9200 4650 9100 4650
-Connection ~ 9100 4650
-Wire Wire Line
-	9100 4450 9100 4650
+	2850 4100 3250 4100
 $Comp
-L power:+5V #PWR?
-U 1 1 61686619
-P 9300 2200
-F 0 "#PWR?" H 9300 2050 50  0001 C CNN
-F 1 "+5V" H 9315 2373 50  0000 C CNN
-F 2 "" H 9300 2200 50  0001 C CNN
-F 3 "" H 9300 2200 50  0001 C CNN
-	1    9300 2200
-	1    0    0    -1
+L Device:LED D1
+U 1 1 616F12B7
+P 2950 5150
+F 0 "D1" H 2943 4895 50  0000 C CNN
+F 1 "LED" H 2943 4986 50  0000 C CNN
+F 2 "" H 2950 5150 50  0001 C CNN
+F 3 "~" H 2950 5150 50  0001 C CNN
+	1    2950 5150
+	-1   0    0    1
+$EndComp
+$Comp
+L Device:LED D2
+U 1 1 616F1A83
+P 2700 4800
+F 0 "D2" H 2693 4545 50  0000 C CNN
+F 1 "LED" H 2693 4636 50  0000 C CNN
+F 2 "" H 2700 4800 50  0001 C CNN
+F 3 "~" H 2700 4800 50  0001 C CNN
+	1    2700 4800
+	-1   0    0    1
 $EndComp
 Wire Wire Line
-	9300 2200 9300 2350
+	2800 4450 2000 4450
 $Comp
-L Switch:SW_Push SW?
-U 1 1 61686626
-P 10350 3450
-F 0 "SW?" H 10350 3735 50  0000 C CNN
-F 1 "SW_Push" H 10350 3644 50  0000 C CNN
-F 2 "" H 10350 3650 50  0001 C CNN
-F 3 "~" H 10350 3650 50  0001 C CNN
-	1    10350 3450
-	-1   0    0    -1
+L Device:LED D3
+U 1 1 616F25D0
+P 2950 4450
+F 0 "D3" H 2943 4195 50  0000 C CNN
+F 1 "LED" H 2943 4286 50  0000 C CNN
+F 2 "" H 2950 4450 50  0001 C CNN
+F 3 "~" H 2950 4450 50  0001 C CNN
+	1    2950 4450
+	-1   0    0    1
 $EndComp
 $Comp
-L power:GND #PWR?
-U 1 1 6168662C
-P 10650 3600
-F 0 "#PWR?" H 10650 3350 50  0001 C CNN
-F 1 "GND" H 10655 3427 50  0000 C CNN
-F 2 "" H 10650 3600 50  0001 C CNN
-F 3 "" H 10650 3600 50  0001 C CNN
-	1    10650 3600
-	-1   0    0    -1
+L Device:LED D4
+U 1 1 616F2AF9
+P 2700 4100
+F 0 "D4" H 2693 3845 50  0000 C CNN
+F 1 "LED" H 2693 3936 50  0000 C CNN
+F 2 "" H 2700 4100 50  0001 C CNN
+F 3 "~" H 2700 4100 50  0001 C CNN
+	1    2700 4100
+	-1   0    0    1
 $EndComp
-$Comp
-L LED:CQY99 D?
-U 1 1 61686638
-P 7750 4050
-F 0 "D?" H 7700 4340 50  0000 C CNN
-F 1 "CQY99" H 7700 4249 50  0000 C CNN
-F 2 "LED_THT:LED_D5.0mm_IRGrey" H 7750 4225 50  0001 C CNN
-F 3 "https://www.prtice.info/IMG/pdf/CQY99.pdf" H 7700 4050 50  0001 C CNN
-	1    7750 4050
-	1    0    0    -1
-$EndComp
-$Comp
-L Device:R R?
-U 1 1 6168664A
-P 8200 4050
-F 0 "R?" V 7993 4050 50  0000 C CNN
-F 1 "510" V 8084 4050 50  0000 C CNN
-F 2 "" V 8130 4050 50  0001 C CNN
-F 3 "~" H 8200 4050 50  0001 C CNN
-	1    8200 4050
-	0    1    1    0
-$EndComp
-$Comp
-L power:GND #PWR?
-U 1 1 61686669
-P 7350 4150
-F 0 "#PWR?" H 7350 3900 50  0001 C CNN
-F 1 "GND" H 7355 3977 50  0000 C CNN
-F 2 "" H 7350 4150 50  0001 C CNN
-F 3 "" H 7350 4150 50  0001 C CNN
-	1    7350 4150
-	1    0    0    -1
-$EndComp
-Wire Wire Line
-	9600 3450 10150 3450
-Wire Wire Line
-	10550 3450 10650 3450
-Wire Wire Line
-	10650 3450 10650 3600
-Wire Wire Line
-	8350 4050 8600 4050
-Wire Wire Line
-	8050 4050 7850 4050
-Wire Wire Line
-	7550 4050 7350 4050
-Wire Wire Line
-	7350 4050 7350 4150
 $EndSCHEMATC
