File: Labs/05-segment/KitchenAlarm/KitchenAlarm.sch (KiCad schematic (older format))
At the start: 9 parts, among them SW1 SW_Push, SW2 SW_Push, SW3 SW_Push, U1 CA56-12EWA, U2 74HC595, U3 74HC595

Commit message: scheme
Connections:
- net +5V: now also U2.16 (VCC), U3.16 (VCC)
- net GND: now also U2.8 (GND), U3.8 (GND)
Changed lines of the file:
@@
 Wire Wire Line
 	2550 4600 3700 4600
+$Comp
+L power:+5V #PWR?
+U 1 1 61766F4A
+P 2200 1100
+F 0 "#PWR?" H 2200 950 50  0001 C CNN
+F 1 "+5V" H 2215 1273 50  0000 C CNN
+F 2 "" H 2200 1100 50  0001 C CNN
+F 3 "" H 2200 1100 50  0001 C CNN
+	1    2200 1100
+	1    0    0    -1
+$EndComp
+$Comp
+L power:+5V #PWR?
+U 1 1 61767AA4
+P 3850 1100
+F 0 "#PWR?" H 3850 950 50  0001 C CNN
+F 1 "+5V" H 3865 1273 50  0000 C CNN
+F 2 "" H 3850 1100 50  0001 C CNN
+F 3 "" H 3850 1100 50  0001 C CNN
+	1    3850 1100
+	1    0    0    -1
+$EndComp
+$Comp
+L power:GND #PWR?
+U 1 1 61768151
+P 2200 2750
+F 0 "#PWR?" H 2200 2500 50  0001 C CNN
+F 1 "GND" H 2205 2577 50  0000 C CNN
+F 2 "" H 2200 2750 50  0001 C CNN
+F 3 "" H 2200 2750 50  0001 C CNN
+	1    2200 2750
+	1    0    0    -1
+$EndComp
+$Comp
+L power:GND #PWR?
+U 1 1 61768798
+P 3850 2750
+F 0 "#PWR?" H 3850 2500 50  0001 C CNN
+F 1 "GND" H 3855 2577 50  0000 C CNN
+F 2 "" H 3850 2750 50  0001 C CNN
+F 3 "" H 3850 2750 50  0001 C CNN
+	1    3850 2750
+	1    0    0    -1
+$EndComp
+Wire Wire Line
+	3850 2750 3850 2650
+Wire Wire Line
+	2200 2750 2200 2650
+Wire Wire Line
+	2200 1350 2200 1100
+Wire Wire Line
+	3850 1350 3850 1100
 $EndSCHEMATC
