File: Labs/06-lcd/KitchenAlarm/KitchenAlarm/KitchenAlarm.sch (KiCad schematic (older format))
At the start: 6 parts

Commit message: readme
Parts:
- added U?: HD44780, Display:LM16255, symbol Display_Character:LM16255K
- R?: value R -> 1k
Connections:
- net GND: now also U?.1 (VSS), U?.5 (R/W)
- net VCC: now also U?.2 (VDD)
- net at A?.17 (D2): now also U?.4 (RS)
- net at A?.18 (D3): now also U?.6 (E)
- net at A?.19 (D4): now also U?.11 (DB4)
- net at A?.20 (D5): now also U?.12 (DB5)
- net at A?.21 (D6): now also U?.13 (DB6)
- net at A?.22 (D7): now also U?.14 (DB7)
- no-connect marks 0 -> 5
Changed lines of the file:
@@
 P 3250 5000
 F 0 "R?" H 3180 4954 50  0000 R CNN
-F 1 "R" H 3180 5045 50  0000 R CNN
+F 1 "1k" H 3180 5045 50  0000 R CNN
 F 2 "" V 3180 5000 50  0001 C CNN
 F 3 "~" H 3250 5000 50  0001 C CNN
@@
 Wire Wire Line
 	1850 5350 1850 4950
+$Comp
+L Display_Character:LM16255K U?
+U 1 1 617A40CF
+P 2200 2450
+F 0 "U?" V 2250 1550 50  0000 R CNN
+F 1 "HD44780" V 2150 1550 50  0000 R CNN
+F 2 "Display:LM16255" H 2200 1650 50  0001 C CNN
+F 3 "http://pdf.datasheetcatalog.com/datasheet/Sharp/mXvtrzw.pdf" H 2300 2350 50  0001 C CNN
+	1    2200 2450
+	0    -1   -1   0
+$EndComp
+$Comp
+L power:VCC #PWR?
+U 1 1 617A5D0E
+P 1400 2400
+F 0 "#PWR?" H 1400 2250 50  0001 C CNN
+F 1 "VCC" H 1415 2573 50  0000 C CNN
+F 2 "" H 1400 2400 50  0001 C CNN
+F 3 "" H 1400 2400 50  0001 C CNN
+	1    1400 2400
+	1    0    0    -1
+$EndComp
+Wire Wire Line
+	1500 2450 1400 2450
+Wire Wire Line
+	1400 2450 1400 2400
+$Comp
+L power:GND #PWR?
+U 1 1 617A67FB
+P 1800 2950
+F 0 "#PWR?" H 1800 2700 50  0001 C CNN
+F 1 "GND" H 1805 2777 50  0000 C CNN
+F 2 "" H 1800 2950 50  0001 C CNN
+F 3 "" H 1800 2950 50  0001 C CNN
+	1    1800 2950
+	1    0    0    -1
+$EndComp
+$Comp
+L power:GND #PWR?
+U 1 1 617A75A6
+P 3050 2550
+F 0 "#PWR?" H 3050 2300 50  0001 C CNN
+F 1 "GND" H 3055 2377 50  0000 C CNN
+F 2 "" H 3050 2550 50  0001 C CNN
+F 3 "" H 3050 2550 50  0001 C CNN
+	1    3050 2550
+	1    0    0    -1
+$EndComp
+Wire Wire Line
+	1800 2950 1800 2850
+Wire Wire Line
+	3050 2550 3050 2450
+Wire Wire Line
+	3050 2450 2900 2450
+Wire Wire Line
+	3450 4150 2700 4150
+Wire Wire Line
+	2700 4150 2700 2850
+Wire Wire Line
+	3450 4050 2600 4050
+Wire Wire Line
+	2600 4050 2600 2850
+Wire Wire Line
+	3450 3950 2500 3950
+Wire Wire Line
+	2500 3950 2500 2850
+Wire Wire Line
+	3450 3850 2400 3850
+Wire Wire Line
+	2400 3850 2400 2850
+Wire Wire Line
+	1700 2850 1700 3650
+Wire Wire Line
+	1700 3650 3450 3650
+Wire Wire Line
+	3450 3750 1900 3750
+Wire Wire Line
+	1900 3750 1900 2850
+NoConn ~ 2000 2050
+NoConn ~ 2000 2850
+NoConn ~ 2100 2850
+NoConn ~ 2200 2850
+NoConn ~ 2300 2850
 $EndSCHEMATC

Commit message: kitchenAlarm
Parts:
- added RV1: R_POT, symbol Device:R_POT
- gave numbers to parts that had none: 7
Connections:
- net GND: now also RV1.1
- net VCC: now also RV1.3
- net at U1.3 (VO): now also RV1.2
- no-connect marks 5 -> 4
Changed lines of the file:
@@
 $EndDescr
 $Comp
-L MCU_Module:Arduino_UNO_R3 A?
+L MCU_Module:Arduino_UNO_R3 A1
 U 1 1 617988E7
 P 3950 4050
-F 0 "A?" H 3950 5231 50  0000 C CNN
+F 0 "A1" H 3950 5231 50  0000 C CNN
 F 1 "Arduino_UNO_R3" H 3950 5140 50  0000 C CNN
 F 2 "Module:Arduino_UNO_R3" H 3950 4050 50  0001 C CIN
@@
 $EndComp
 $Comp
-L Switch:SW_Push SW?
+L Switch:SW_Push SW3
 U 1 1 61799A9C
 P 2200 5350
-F 0 "SW?" H 2200 5635 50  0000 C CNN
+F 0 "SW3" H 2200 5635 50  0000 C CNN
 F 1 "SW_Push" H 2200 5544 50  0000 C CNN
 F 2 "" H 2200 5550 50  0001 C CNN
@@
 $EndComp
 $Comp
-L Device:LED D?
+L Device:LED D1
 U 1 1 6179A0BC
 P 3250 5450
-F 0 "D?" V 3289 5332 50  0000 R CNN
+F 0 "D1" V 3289 5332 50  0000 R CNN
 F 1 "LED" V 3198 5332 50  0000 R CNN
 F 2 "" H 3250 5450 50  0001 C CNN
@@
 $EndComp
 $Comp
-L Device:R R?
+L Device:R R1
 U 1 1 6179A891
 P 3250 5000
-F 0 "R?" H 3180 4954 50  0000 R CNN
+F 0 "R1" H 3180 4954 50  0000 R CNN
 F 1 "1k" H 3180 5045 50  0000 R CNN
 F 2 "" V 3180 5000 50  0001 C CNN
@@
 $EndComp
 $Comp
-L Switch:SW_Push SW?
+L Switch:SW_Push SW2
 U 1 1 6179F586
 P 2150 4950
-F 0 "SW?" H 2150 5235 50  0000 C CNN
+F 0 "SW2" H 2150 5235 50  0000 C CNN
 F 1 "SW_Push" H 2150 5144 50  0000 C CNN
 F 2 "" H 2150 5150 50  0001 C CNN
@@
 $EndComp
 $Comp
-L Switch:SW_Push SW?
+L Switch:SW_Push SW1
 U 1 1 6179F7B1
 P 2150 4550
-F 0 "SW?" H 2150 4835 50  0000 C CNN
+F 0 "SW1" H 2150 4835 50  0000 C CNN
 F 1 "SW_Push" H 2150 4744 50  0000 C CNN
 F 2 "" H 2150 4750 50  0001 C CNN
@@
 $EndComp
 $Comp
-L power:GND #PWR?
+L power:GND #PWR07
 U 1 1 6179FB8E
 P 3950 5950
-F 0 "#PWR?" H 3950 5700 50  0001 C CNN
+F 0 "#PWR07" H 3950 5700 50  0001 C CNN
 F 1 "GND" H 3955 5777 50  0000 C CNN
 F 2 "" H 3950 5950 50  0001 C CNN
@@
 $EndComp
 $Comp
-L power:VCC #PWR?
+L power:VCC #PWR05
 U 1 1 617A03D8
 P 4150 2750
-F 0 "#PWR?" H 4150 2600 50  0001 C CNN
+F 0 "#PWR05" H 4150 2600 50  0001 C CNN
 F 1 "VCC" H 4165 2923 50  0000 C CNN
 F 2 "" H 4150 2750 50  0001 C CNN
@@
 	1850 5350 1850 4950
 $Comp
-L Display_Character:LM16255K U?
+L Display_Character:LM16255K U1
 U 1 1 617A40CF
 P 2200 2450
-F 0 "U?" V 2250 1550 50  0000 R CNN
+F 0 "U1" V 2250 1550 50  0000 R CNN
 F 1 "HD44780" V 2150 1550 50  0000 R CNN
 F 2 "Display:LM16255" H 2200 1650 50  0001 C CNN
@@
 $EndComp
 $Comp
-L power:VCC #PWR?
+L power:VCC #PWR03
 U 1 1 617A5D0E
 P 1400 2400
-F 0 "#PWR?" H 1400 2250 50  0001 C CNN
+F 0 "#PWR03" H 1400 2250 50  0001 C CNN
 F 1 "VCC" H 1415 2573 50  0000 C CNN
 F 2 "" H 1400 2400 50  0001 C CNN
@@
 	1400 2450 1400 2400
 $Comp
-L power:GND #PWR?
+L power:GND #PWR06
 U 1 1 617A67FB
 P 1800 2950
-F 0 "#PWR?" H 1800 2700 50  0001 C CNN
+F 0 "#PWR06" H 1800 2700 50  0001 C CNN
 F 1 "GND" H 1805 2777 50  0000 C CNN
 F 2 "" H 1800 2950 50  0001 C CNN
@@
 $EndComp
 $Comp
-L power:GND #PWR?
+L power:GND #PWR04
 U 1 1 617A75A6
 P 3050 2550
-F 0 "#PWR?" H 3050 2300 50  0001 C CNN
+F 0 "#PWR04" H 3050 2300 50  0001 C CNN
 F 1 "GND" H 3055 2377 50  0000 C CNN
 F 2 "" H 3050 2550 50  0001 C CNN
@@
 Wire Wire Line
 	1900 3750 1900 2850
-NoConn ~ 2000 2050
 NoConn ~ 2000 2850
 NoConn ~ 2100 2850
 NoConn ~ 2200 2850
 NoConn ~ 2300 2850
+$Comp
+L Device:R_POT RV1
+U 1 1 61815299
+P 2000 1750
+F 0 "RV1" V 1793 1750 50  0000 C CNN
+F 1 "R_POT" V 1884 1750 50  0000 C CNN
+F 2 "" H 2000 1750 50  0001 C CNN
+F 3 "~" H 2000 1750 50  0001 C CNN
+	1    2000 1750
+	0    1    1    0
+$EndComp
+Wire Wire Line
+	2000 2050 2000 1900
+$Comp
+L power:VCC #PWR01
+U 1 1 61817132
+P 1700 1650
+F 0 "#PWR01" H 1700 1500 50  0001 C CNN
+F 1 "VCC" H 1715 1823 50  0000 C CNN
+F 2 "" H 1700 1650 50  0001 C CNN
+F 3 "" H 1700 1650 50  0001 C CNN
+	1    1700 1650
+	1    0    0    -1
+$EndComp
+$Comp
+L power:GND #PWR02
+U 1 1 6181758A
+P 2300 1850
+F 0 "#PWR02" H 2300 1600 50  0001 C CNN
+F 1 "GND" H 2305 1677 50  0000 C CNN
+F 2 "" H 2300 1850 50  0001 C CNN
+F 3 "" H 2300 1850 50  0001 C CNN
+	1    2300 1850
+	1    0    0    -1
+$EndComp
+Wire Wire Line
+	1700 1650 1700 1750
+Wire Wire Line
+	1700 1750 1850 1750
+Wire Wire Line
+	2150 1750 2300 1750
+Wire Wire Line
+	2300 1750 2300 1850
 $EndSCHEMATC
