File: Labs/07-uart/TemperatureMeter/TemperatureMeter/TemperatureMeter.sch (KiCad schematic (older format))
At the start: 9 parts, among them Q1 9013, SW1 SW_Push, U1 TC1046

Commit message: readme
Parts:
- LCD1: symbol arduino_lcd:DS1 -> TemperatureMeter-rescue:DS1-arduino_lcd
Changed lines of the file:
@@
 $EndComp
 $Comp
-L arduino_lcd:DS1 LCD1
+L TemperatureMeter-rescue:DS1-arduino_lcd LCD1
 U 1 1 618493AF
 P 5950 2100
