File: Labs/08-i2c/ArduinoUno/ArduinoUno/ArduinoUno.sch (KiCad schematic (older format))
At the start: 1 part

Commit message: i2c, new arduino picture
Connections:
- net INT: no longer A1.20 (D5), A1.21 (D6)
- new net PWM0: A1.20 (D5), A1.21 (D6)
Changed lines of the file:
@@
 $EndDescr
 Text GLabel 1550 4300 0    50   Input ~ 0
-PWM
+PWM2
 Text GLabel 2000 4500 0    50   Input ~ 0
-PWM
+PWM0
 Text GLabel 2000 4600 0    50   Input ~ 0
-PWM
+PWM0
 Text GLabel 1550 5100 0    50   Input ~ 0
-PWM
+PWM2
 Text GLabel 1550 4900 0    50   Input ~ 0
-PWM
+PWM1
 Text GLabel 2000 4900 0    50   Input ~ 0
-PWM
+PWM1
 Text GLabel 3600 4600 2    50   Input ~ 0
 ADC
@@
 Wire Wire Line
 	2250 4900 2000 4900
-Wire Wire Line
-	2250 5000 1750 5000
-Wire Wire Line
-	1750 5000 1750 4900
-Wire Wire Line
-	1750 4900 1550 4900
 Wire Wire Line
 	2250 5100 1750 5100
@@
 	3900 5100 4050 5100
 Wire Wire Line
-	1750 5000 1550 5000
-Connection ~ 1750 5000
-Wire Wire Line
 	1550 5200 1750 5200
 Wire Wire Line
@@
 F1 "file618C7E80.sch" 50
 $EndSheet
+Wire Wire Line
+	1550 5000 1650 5000
+Wire Wire Line
+	1550 4900 1650 4900
+Wire Wire Line
+	1650 4900 1650 5000
+Connection ~ 1650 5000
+Wire Wire Line
+	1650 5000 2250 5000
 $EndSCHEMATC
